File: left/pcb-flat-left.kicad_pcb (KiCad board)
At the start: 2 copper layers, 225.3 x 231.1 mm, 116 parts, among them J1 DB15_Female, SW1 MX-NO-LED, SW10 MX-NO-LED, SW11 MX-NO-LED, SW12 MX-NO-LED, SW13 MX-NO-LED, SW14 MX-NO-LED, SW15 MX-NO-LED, SW16 MX-NO-LED, SW17 MX-NO-LED, SW18 MX-NO-LED, SW19 MX-NO-LED, SW2 MX-NO-LED, SW20 MX-NO-LED, SW21 MX-NO-LED, SW22 MX-NO-LED, SW23 MX-NO-LED, SW24 MX-NO-LED, SW25 MX-NO-LED, SW26 MX-NO-LED, SW27 MX-NO-LED, SW28 MX-NO-LED, SW29 MX-NO-LED, SW3 MX-NO-LED, SW30 MX-NO-LED, SW31 MX-NO-LED, SW32 MX-NO-LED, SW33 MX-NO-LED, SW34 MX-NO-LED, SW35 MX-NO-LED, SW36 MX-NO-LED, SW37 MX-NO-LED, SW38 MX-NO-LED, SW39 MX-NO-LED, SW4 MX-NO-LED, SW40 MX-NO-LED, SW41 MX-NO-LED, SW42 MX-NO-LED, SW43 MX-NO-LED, SW44 MX-NO-LED, SW45 MX-NO-LED, SW46 MX-NO-LED, SW47 MX-NO-LED, SW5 MX-NO-LED, SW6 MX-NO-LED, SW7 MX-NO-LED, SW8 MX-NO-LED, SW9 MX-NO-LED, U1 Teensy++2.0_(Arduino)

Commit message: updated files
Parts:
- removed the REF** at (59.2, 264.5)
- removed the REF** at (60.3, 248.4) (x2)
- removed the REF** at (59.0, 264.6)
- added REF**: OSHW-Logo2_24.3x20mm_SilkScreen, Symbol:OSHW-Logo2_24.3x20mm_SilkScreen, B.Cu at (187.7, 261.3)
- added REF**: OSHW-Logo2_24.3x20mm_SilkScreen, Symbol:OSHW-Logo2_24.3x20mm_SilkScreen, F.Cu at (187.7, 261.2)
- added REF**: KiCad-Logo2_20mm_SilkScreen, Symbol:KiCad-Logo2_20mm_SilkScreen, B.Cu at (79.4, 256.6)
- added REF**: KiCad-Logo2_20mm_SilkScreen, Symbol:KiCad-Logo2_20mm_SilkScreen, F.Cu at (79.6, 256.5)
- J1: footprint Connector_Dsub:DSUB-15-HD_Female_Horizontal_P2.29x1.98mm_EdgePinOffset9.40mm -> Connector_Dsub:DSUB-15-HD_Female_Horizontal_P2.29x1.98mm_EdgePinOffset8.35mm_Housed_MountingHolesOffset10.89mm
- moved D47 18.9 mm to (200.7, 228.8)
- moved D46 18.9 mm to (206.1, 204.4)
- moved SW46 18.9 mm to (208.0, 214.5)
- moved SW47 18.9 mm to (228.6, 226.3)
- moved SW45 18.9 mm to (219.8, 193.9)
- moved D48 18.8 mm to (221.5, 240.7)
- moved SW44 18.7 mm to (187.3, 202.6)
- moved D45 18.3 mm to (179.9, 217.0)
- moved J1 1.50 mm to (232.5, 197.2)
Connections:
- D45 pad 1: ArrowsC -> COL5+6
- D46 pad 1: ArrowsC -> Arrow-Left
- D47 pad 1: ArrowsC -> COL7+8
- D48 pad 1: ArrowsC -> Arrow-Left
- J1 pad 1: ROW1+2ext -> ROW1ext
- J1 pad 10: Net-(J1-Pad10) -> ROW4ext
- J1 pad 11: Net-(J1-Pad11) -> ROW6ext
- J1 pad 13: Net-(J1-Pad13) -> COL1+2ext
- J1 pad 14: Net-(J1-Pad14) -> COL5+6ext
- J1 pad 2: ROW3+4ext -> ROW3ext
- J1 pad 3: ROW5+6ext -> ROW5ext
- J1 pad 4: COL1+2ext -> Net-(J1-Pad4)
- J1 pad 5: COL3+4ext -> Net-(J1-Pad5)
- J1 pad 6: COL5+6ext -> COL3+4ext
- J1 pad 8: ArrowsRext -> Arrow-Right
- J1 pad 9: ArrowsCext -> ROW2ext
- SW1 pad 1: ROW1+2 -> ROW1
- SW10 pad 1: ROW5+6 -> ROW5
- SW11 pad 1: ROW3+4 -> ROW4
- SW12 pad 1: ROW5+6 -> ROW6
- SW13 pad 1: ROW1+2 -> ROW1
- SW14 pad 1: ROW1+2 -> ROW2
- SW15 pad 1: ROW3+4 -> ROW3
- SW16 pad 1: ROW5+6 -> ROW5
- SW17 pad 1: ROW3+4 -> ROW4
- SW18 pad 1: ROW5+6 -> ROW6
- SW19 pad 1: ROW1+2 -> ROW1
- SW2 pad 1: ROW1+2 -> ROW2
- SW20 pad 1: ROW1+2 -> ROW2
- SW21 pad 1: ROW3+4 -> ROW3
- SW22 pad 1: ROW5+6 -> ROW5
- SW23 pad 1: ROW3+4 -> ROW4
- SW24 pad 1: ROW5+6 -> ROW6
- SW25 pad 1: ROW1+2 -> ROW1
- SW26 pad 1: ROW1+2 -> ROW2
- SW27 pad 1: ROW3+4 -> ROW3
- SW28 pad 1: ROW5+6 -> ROW5
- SW29 pad 1: ROW3+4 -> ROW4
- SW3 pad 1: ROW3+4 -> ROW3
- SW30 pad 1: ROW5+6 -> ROW6
- SW31 pad 1: ROW1+2 -> ROW1
- SW32 pad 1: ROW1+2 -> ROW2
- SW33 pad 1: ROW3+4 -> ROW3
- SW34 pad 1: ROW5+6 -> ROW5
- SW35 pad 1: ROW3+4 -> ROW4
- SW36 pad 1: ROW1+2 -> ROW1
- SW37 pad 1: ROW1+2 -> ROW2
- SW38 pad 1: ROW3+4 -> ROW3
- SW39 pad 1: ROW5+6 -> ROW5
- SW4 pad 1: ROW5+6 -> ROW5
- SW40 pad 1: ROW3+4 -> ROW4
- SW41 pad 1: ROW1+2 -> ROW2
- SW42 pad 1: ROW3+4 -> ROW3
- SW43 pad 1: ROW5+6 -> ROW5
- SW44 pad 1: ArrowsR -> ROW6
- SW45 pad 1: ArrowsR -> ROW5
- SW46 pad 1: ArrowsR -> ROW6
- SW47 pad 1: ArrowsR -> ROW6
- SW5 pad 1: ROW3+4 -> ROW4
- SW6 pad 1: ROW5+6 -> ROW6
- SW7 pad 1: ROW1+2 -> ROW1
- SW8 pad 1: ROW1+2 -> ROW2
- SW9 pad 1: ROW3+4 -> ROW3
- U1 pad 10: Net-(U1-Pad10) -> ROW3
- U1 pad 11: Net-(U1-Pad11) -> ROW4
- U1 pad 12: ArrowsCext -> ROW5
- U1 pad 13: ArrowsRext -> ROW6
- U1 pad 14: COL7+8ext -> ROW1ext
- U1 pad 15: COL5+6ext -> ROW2ext
- U1 pad 16: COL3+4ext -> ROW3ext
- U1 pad 20: Net-(U1-Pad20) -> Arrow-Left
- U1 pad 24: Net-(U1-Pad24) -> ROW4ext
- U1 pad 29: ROW5+6 -> Arrow-Right
- U1 pad 3: Net-(U1-Pad3) -> COL1+2ext
- U1 pad 30: ROW3+4 -> Net-(U1-Pad30)
- U1 pad 31: ROW1+2 -> Net-(U1-Pad31)
- U1 pad 36: ROW1+2ext -> Net-(U1-Pad36)
- U1 pad 37: ROW3+4ext -> ROW5ext
- U1 pad 38: ROW5+6ext -> ROW6ext
- U1 pad 4: Net-(U1-Pad4) -> COL3+4ext
- U1 pad 5: Net-(U1-Pad5) -> COL5+6ext
- U1 pad 6: Net-(U1-Pad6) -> COL7+8ext
- U1 pad 7: ArrowsC -> ROW1
- U1 pad 8: ArrowsR -> ROW2
Routing:
- net ROW1+2: track 511.8 -> 0.00 mm
- net ROW3+4: track 427.9 -> 0.00 mm
- net ROW1: track 0.00 -> 336.4 mm
- net ROW5+6: track 331.4 -> 0.00 mm
- net ROW2: track 0.00 -> 309.6 mm
- net ROW3: track 0.00 -> 292.9 mm
- net ROW5: track 0.00 -> 262.8 mm
- net ROW4: track 0.00 -> 235.1 mm
- net ArrowsC: track 234.8 -> 0.00 mm
- net ROW6: track 0.00 -> 228.1 mm, vias 0 -> 1
- net ROW5ext: track 0.00 -> 225.7 mm
- net ROW6ext: track 0.00 -> 218.6 mm
- net ArrowsCext: track 218.3 -> 0.00 mm
- net ArrowsR: track 216.0 -> 0.00 mm, vias 1 -> 0
- net ROW5+6ext: track 214.7 -> 0.00 mm
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Other:
- board text added: "https://github.com/Supermagnum/98keys-ergo/"

Commit message: Add files via upload
updated files
Parts:
- J1: value DB15_Female -> 5745783-4; footprint Connector_Dsub:DSUB-15-HD_Female_Horizontal_P2.29x1.98mm_EdgePinOffset8.35mm_Housed_MountingHolesOffset10.89mm -> Connector_Dsub:DSUB-25_Female_Horizontal_P2.77x2.84mm_EdgePinOffset7.70mm_Housed_MountingHolesOffset9.12mm
- moved J1 13.4 mm to (235.3, 210.3)
Connections:
- D1 pad 1: COL1+2 -> COL1
- D10 pad 1: COL1+2 -> COL2
- D11 pad 1: COL1+2 -> COL2
- D12 pad 1: COL1+2 -> COL2
- D14 pad 1: COL3+4 -> COL3
- D15 pad 1: COL3+4 -> COL3
- D16 pad 1: COL3+4 -> COL3
- D17 pad 1: COL3+4 -> COL3
- D18 pad 1: COL3+4 -> COL3
- D19 pad 1: COL3+4 -> COL3
- D2 pad 1: COL1+2 -> COL1
- D20 pad 1: COL3+4 -> COL4
- D21 pad 1: COL3+4 -> COL4
- D22 pad 1: COL3+4 -> COL4
- D23 pad 1: COL3+4 -> COL4
- D24 pad 1: COL3+4 -> COL4
- D25 pad 1: COL3+4 -> COL4
- D26 pad 1: COL5+6 -> COL5
- D27 pad 1: COL5+6 -> COL5
- D28 pad 1: COL5+6 -> COL5
- D29 pad 1: COL5+6 -> COL5
- D3 pad 1: COL1+2 -> COL1
- D30 pad 1: COL5+6 -> COL5
- D31 pad 1: COL5+6 -> COL5
- D32 pad 1: COL5+6 -> COL6
- D33 pad 1: COL5+6 -> COL6
- D34 pad 1: COL5+6 -> COL6
- D35 pad 1: COL5+6 -> COL6
- D36 pad 1: COL5+6 -> COL6
- D37 pad 1: COL7+8 -> COL7
- D38 pad 1: COL7+8 -> COL7
- D39 pad 1: COL7+8 -> COL7
- D4 pad 1: COL1+2 -> COL1
- D40 pad 1: COL7+8 -> COL7
- D41 pad 1: COL7+8 -> COL7
- D42 pad 1: COL7+8 -> COL8
- D43 pad 1: COL7+8 -> COL8
- D44 pad 1: COL7+8 -> COL8
- D45 pad 1: COL5+6 -> COL6
- D47 pad 1: COL7+8 -> COL8
- D5 pad 1: COL1+2 -> COL1
- D6 pad 1: COL1+2 -> COL1
- D7 pad 1: COL1+2 -> COL2
- D8 pad 1: COL1+2 -> COL2
- D9 pad 1: COL1+2 -> COL2
- J1 pad 0: (no net) -> GND
- J1 pad 10: ROW4ext -> Net-(J1-Pad10)
- J1 pad 11: ROW6ext -> Net-(J1-Pad11)
- J1 pad 13: COL1+2ext -> Net-(J1-Pad13)
- J1 pad 14: COL5+6ext -> ROW2ext
- J1 pad 15: GND -> ROW4ext
- J1 pad 4: Net-(J1-Pad4) -> COL1x
- J1 pad 5: Net-(J1-Pad5) -> COL3x
- J1 pad 6: COL3+4ext -> COL5x
- J1 pad 7: COL7+8ext -> COL7x
- J1 pad 9: ROW2ext -> Net-(J1-Pad9)
- U1 pad 25: COL7+8 -> COL5
- U1 pad 26: COL5+6 -> COL6
- U1 pad 27: COL3+4 -> COL7
- U1 pad 28: COL1+2 -> COL8
- U1 pad 3: COL1+2ext -> COL1
- U1 pad 30: Net-(U1-Pad30) -> ROW6
- U1 pad 31: Net-(U1-Pad31) -> ROW5
- U1 pad 34: Net-(U1-Pad34) -> COL8x
- U1 pad 35: Net-(U1-Pad35) -> COL7x
- U1 pad 36: Net-(U1-Pad36) -> COL6x
- U1 pad 37: ROW5ext -> COL5x
- U1 pad 38: ROW6ext -> COL4x
- U1 pad 39: COL1+2ext -> COL3x
- U1 pad 4: COL3+4ext -> COL2
- U1 pad 40: Net-(U1-Pad40) -> COL1x
- U1 pad 41: Net-(U1-Pad41) -> COL2x
- U1 pad 42: Net-(U1-Pad42) -> ROW5ext
- U1 pad 47: Net-(U1-Pad47) -> ROW6ext
- U1 pad 5: COL5+6ext -> COL3
- U1 pad 6: COL7+8ext -> COL4
Routing:
- net COL5+6: track 393.3 -> 0.00 mm
- net COL7+8: track 385.1 -> 0.00 mm
- net COL3+4: track 326.1 -> 0.00 mm
- net COL8: track 0.00 -> 303.5 mm
- net COL6: track 0.00 -> 279.3 mm
- net COL1+2: track 271.2 -> 0.00 mm
- net COL7: track 0.00 -> 268.2 mm, vias 0 -> 1
- net COL1+2ext: track 265.9 -> 0.00 mm
- net COL6x: track 0.00 -> 239.2 mm
- net COL4x: track 0.00 -> 229.2 mm
- net COL2x: track 0.00 -> 229.1 mm
- net COL1x: track 0.00 -> 221.4 mm
- net COL4: track 0.00 -> 220.2 mm
- net COL5: track 0.00 -> 219.8 mm
- net COL3x: track 0.00 -> 219.8 mm
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Other:
- net class Front added: clearance 0.15, trace_width 0.25, via_dia 0.8, via_drill 0.4
- net class back added: clearance 0.15, trace_width 0.25, via_dia 0.8, via_drill 0.4
