File: left/pcb-flat-left.sch (KiCad schematic (older format))
At the start: 112 parts, among them J1 DB15_Female, SW1 MX-NO-LED, SW10 MX-NO-LED, SW11 MX-NO-LED, SW12 MX-NO-LED, SW13 MX-NO-LED, SW14 MX-NO-LED, SW15 MX-NO-LED, SW16 MX-NO-LED, SW17 MX-NO-LED, SW18 MX-NO-LED, SW19 MX-NO-LED, SW2 MX-NO-LED, SW20 MX-NO-LED, SW21 MX-NO-LED, SW22 MX-NO-LED, SW23 MX-NO-LED, SW24 MX-NO-LED, SW25 MX-NO-LED, SW26 MX-NO-LED, SW27 MX-NO-LED, SW28 MX-NO-LED, SW29 MX-NO-LED, SW3 MX-NO-LED, SW30 MX-NO-LED, SW31 MX-NO-LED, SW32 MX-NO-LED, SW33 MX-NO-LED, SW34 MX-NO-LED, SW35 MX-NO-LED, SW36 MX-NO-LED, SW37 MX-NO-LED, SW38 MX-NO-LED, SW39 MX-NO-LED, SW4 MX-NO-LED, SW40 MX-NO-LED, SW41 MX-NO-LED, SW42 MX-NO-LED, SW43 MX-NO-LED, SW44 MX-NO-LED, SW45 MX-NO-LED, SW46 MX-NO-LED, SW47 MX-NO-LED, SW5 MX-NO-LED, SW6 MX-NO-LED, SW7 MX-NO-LED, SW8 MX-NO-LED, SW9 MX-NO-LED, U1 Teensy++2.0_(Arduino)

Commit message: updated files
Parts:
- J1: footprint Connector_Dsub:DSUB-15-HD_Female_Horizontal_P2.29x1.98mm_EdgePinOffset9.40mm -> Connector_Dsub:DSUB-15-HD_Female_Horizontal_P2.29x1.98mm_EdgePinOffset8.35mm_Housed_MountingHolesOffset10.89mm
- SW44: Field4 (none) -> arrow-left
- SW45: Field4 (none) -> arrow-up
- SW46: Field4 (none) -> arrow-down
- SW47: Field4 (none) -> arrow-right
Connections:
- net COL1+2ext: now also J1.13 (P13), U1.3 (0_INT0_PWM); no longer J1.4
- net COL3+4ext: now also J1.6, U1.4 (1_INT1_PWM); no longer J1.5, U1.16 (13)
- net COL5+6: now also D45.1 (K)
- net COL5+6ext: now also J1.14 (P14), U1.5 (2_INT2_RX); no longer J1.6, U1.15 (12)
- net COL7+8: now also D47.1 (K)
- net COL7+8ext: now also U1.6 (3_INT3_TX); no longer U1.14 (11)
- net ROW3: now reaches U1.10 (7)
- net ROW3: now also SW15.1, SW21.1, SW27.1, SW3.1, SW33.1, SW38.1, SW42.1, SW9.1
- net ROW4: now reaches U1.11 (8)
- net ROW4: now also SW11.1, SW17.1, SW23.1, SW29.1, SW35.1, SW40.1, SW5.1
- net Arrow-Left: now reaches U1.20 (17)
- net Arrow-Left: now also D46.1 (K), D48.1 (K)
- net ROW4ext: now reaches U1.24 (45_A7)
- net ROW4ext: now also J1.10 (P10)
- net ROW6ext: now reaches J1.11 (P111)
- net ROW6ext: now also U1.38 (22)
- removed net ArrowsC: D45.1 (K), D46.1 (K), D47.1 (K), D48.1 (K), U1.7 (4)
- net ArrowsCext renamed ROW2ext
- net ROW2ext: now also U1.15 (12); no longer U1.12 (9)
- net ArrowsR renamed ROW6
- net ROW6: now also SW12.1, SW18.1, SW24.1, SW30.1, SW6.1, U1.13 (10); no longer SW45.1, U1.8 (5)
- net ArrowsRext renamed Arrow-Right
- net Arrow-Right: now also U1.29 (40_A2); no longer U1.13 (10)
- net ROW1+2 renamed ROW2
- net ROW2: now also U1.8 (5); no longer SW1.1, SW13.1, SW19.1, SW25.1, SW31.1, SW36.1, SW7.1, U1.31 (38_A0)
- net ROW1+2ext: no longer names the net of U1.36 (20)
- net ROW1+2ext: no longer J1.1
- removed net ROW3+4: SW11.1, SW15.1, SW17.1, SW21.1, SW23.1, SW27.1, SW29.1, SW3.1, SW33.1, SW35.1, SW38.1, SW40.1, SW42.1, SW5.1, SW9.1, U1.30 (39_A1)
- net ROW3+4ext renamed ROW3ext
- net ROW3ext: now also U1.16 (13); no longer U1.37 (21)
- net ROW5+6 renamed ROW5
- net ROW5: now also SW45.1, U1.12 (9); no longer SW12.1, SW18.1, SW24.1, SW30.1, SW6.1, U1.29 (40_A2)
- net ROW5+6ext renamed ROW5ext
- net ROW5ext: now also U1.37 (21); no longer U1.38 (22)
- new net ROW1: SW1.1, SW13.1, SW19.1, SW25.1, SW31.1, SW36.1, SW7.1, U1.7 (4)
- new net ROW1ext: J1.1, U1.14 (11)
- no-connect marks 34 -> 27
Other:
- moved on the sheet: D1, D10, D11, D12, D13, D14, D15, D16, D17, D18, D19, D2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

Commit message: Add files via upload
updated files
Parts:
- removed J1: DB15_Female, Connector_Dsub:DSUB-15-HD_Female_Horizontal_P2.29x1.98mm_EdgePinOffset8.35mm_Housed_MountingHolesOffset10.89mm, symbol Connector:DB15_Female
- added J1: 5745783-4, Connector_Dsub:DSUB-25_Female_Horizontal_P2.77x2.84mm_EdgePinOffset7.70mm_Housed_MountingHolesOffset9.12mm, symbol Connector:DB25_Female_MountingHoles
Connections:
- net Arrow-Right: now also J1.8
- net GND: now also J1.0 (PAD)
- net ROW1ext: now also J1.1
- net ROW2ext: now also J1.14 (P14)
- net ROW3ext: now also J1.2
- net ROW4ext: now also J1.15 (P15)
- net ROW5: now also U1.31 (38_A0)
- net ROW5ext: now also U1.42 (26_PWM), J1.3; no longer U1.37 (21)
- net ROW6: now also U1.30 (39_A1)
- net ROW6ext: now also U1.47 (31), J1.16 (P16); no longer U1.38 (22)
- net COL8x: now reaches U1.34 (18_INT6)
- net COL8x: now also J1.20 (P20)
- net COL7x: now reaches U1.35 (19_INT7)
- net COL7x: now also J1.7
- net COL6x: now reaches U1.36 (20)
- net COL6x: now also J1.19 (P19)
- net COL1x: now reaches U1.40 (24_PWM)
- net COL1x: now also J1.4
- net COL2x: now reaches U1.41 (25_PWM)
- net COL2x: now also J1.17 (P17)
- removed net COL1+2: D1.1 (K), D10.1 (K), D11.1 (K), D12.1 (K), D2.1 (K), D3.1 (K), D4.1 (K), D5.1 (K), D6.1 (K), D7.1 (K), D8.1 (K), D9.1 (K), U1.28 (41_A3)
- net COL1+2ext renamed COL1
- net COL1: now also D1.1 (K), D2.1 (K), D3.1 (K), D4.1 (K), D5.1 (K), D6.1 (K); no longer U1.39 (23)
- removed net COL3+4: D14.1 (K), D15.1 (K), D16.1 (K), D17.1 (K), D18.1 (K), D19.1 (K), D20.1 (K), D21.1 (K), D22.1 (K), D23.1 (K), D24.1 (K), D25.1 (K), U1.27 (42_A4)
- net COL3+4ext renamed COL2
- net COL2: now also D10.1 (K), D11.1 (K), D12.1 (K), D7.1 (K), D8.1 (K), D9.1 (K)
- net COL5+6 renamed COL6
- net COL6: no longer D26.1 (K), D27.1 (K), D28.1 (K), D29.1 (K), D30.1 (K), D31.1 (K)
- net COL5+6ext renamed COL3
- net COL3: now also D14.1 (K), D15.1 (K), D16.1 (K), D17.1 (K), D18.1 (K), D19.1 (K)
- net COL7+8 renamed COL7
- net COL7: now also U1.27 (42_A4); no longer D42.1 (K), D43.1 (K), D44.1 (K), D47.1 (K), U1.25 (44_A6)
- net COL7+8ext renamed COL4
- net COL4: now also D20.1 (K), D21.1 (K), D22.1 (K), D23.1 (K), D24.1 (K), D25.1 (K)
- new net COL3x: J1.5, U1.39 (23)
- new net COL4x: J1.18 (P18), U1.38 (22)
- new net COL5: D26.1 (K), D27.1 (K), D28.1 (K), D29.1 (K), D30.1 (K), D31.1 (K), U1.25 (44_A6)
- new net COL5x: J1.6, U1.37 (21)
- new net COL8: D42.1 (K), D43.1 (K), D44.1 (K), D47.1 (K), U1.28 (41_A3)
- no-connect marks 27 -> 25
