File: right/pcb-flat-right.kicad_pcb (KiCad board)
At the start: 2 copper layers, 225.5 x 231.2 mm, 107 parts, among them J1 DB15_Female, SW1 MX-NO-LED, SW10 MX-NO-LED, SW11 MX-NO-LED, SW12 MX-NO-LED, SW13 MX-NO-LED, SW14 MX-NO-LED, SW15 MX-NO-LED, SW16 MX-NO-LED, SW17 MX-NO-LED, SW18 MX-NO-LED, SW19 MX-NO-LED, SW2 MX-NO-LED, SW20 MX-NO-LED, SW21 MX-NO-LED, SW22 MX-NO-LED, SW23 MX-NO-LED, SW24 MX-NO-LED, SW25 MX-NO-LED, SW26 MX-NO-LED, SW27 MX-NO-LED, SW28 MX-NO-LED, SW29 MX-NO-LED, SW3 MX-NO-LED, SW30 MX-NO-LED, SW31 MX-NO-LED, SW32 MX-NO-LED, SW33 MX-NO-LED, SW34 MX-NO-LED, SW35 MX-NO-LED, SW36 MX-NO-LED, SW37 MX-NO-LED, SW38 MX-NO-LED, SW39 MX-NO-LED, SW4 MX-NO-LED, SW40 MX-NO-LED, SW41 MX-NO-LED, SW42 MX-NO-LED, SW43 MX-NO-LED, SW44 MX-NO-LED, SW45 MX-NO-LED, SW46 MX-NO-LED, SW47 MX-NO-LED, SW5 MX-NO-LED, SW6 MX-NO-LED, SW7 MX-NO-LED, SW8 MX-NO-LED, SW9 MX-NO-LED

Commit message: updated files, right side.
Parts:
- removed the REF** at (203.5, 224.1)
- removed the REF** at (203.6, 224.1)
- removed the REF** at (203.6, 242.5)
- removed the REF** at (203.6, 242.2)
- added REF**: KiCad-Logo2_20mm_SilkScreen, Symbol:KiCad-Logo2_20mm_SilkScreen, B.Cu at (93.7, 238.4)
- added REF**: KiCad-Logo2_20mm_SilkScreen, Symbol:KiCad-Logo2_20mm_SilkScreen, F.Cu at (93.8, 238.3)
- added REF**: OSHW-Logo2_24.3x20mm_SilkScreen, Symbol:OSHW-Logo2_24.3x20mm_SilkScreen, B.Cu at (191.4, 242.4)
- added REF**: OSHW-Logo2_24.3x20mm_SilkScreen, Symbol:OSHW-Logo2_24.3x20mm_SilkScreen, F.Cu at (191.4, 242.5)
- J1: footprint Connector_Dsub:DSUB-15_Female_Horizontal_P2.77x2.84mm_EdgePinOffset9.40mm -> Connector_Dsub:DSUB-15-HD_Female_Horizontal_P2.29x1.98mm_EdgePinOffset3.03mm_Housed_MountingHolesOffset4.94mm
- moved D46 19.1 mm to (57.4, 189.3)
- moved SW45 19.1 mm to (55.1, 172.2)
- moved D45 19.0 mm to (48.5, 221.9)
- moved SW44 19.0 mm to (46.4, 204.8)
- moved D47 18.9 mm to (69.0, 210.1)
- moved SW46 18.9 mm to (66.9, 193.0)
- moved D48 18.9 mm to (90.1, 197.9)
- moved SW47 18.9 mm to (87.6, 181.0)
- moved J1 14.8 mm to (32.7, 192.5)
Connections:
- D45 pad 1: arrowsC -> COL5+6
- D46 pad 1: arrowsC -> Arrow-Right
- D47 pad 1: arrowsC -> COL7+8
- D48 pad 1: arrowsC -> Arrow-Right
- J1 pad 1: /ROW1+2 -> ROW1
- J1 pad 10: (no net) -> ROW4
- J1 pad 11: (no net) -> ROW6
- J1 pad 12: (no net) -> Net-(J1-Pad12)
- J1 pad 13: (no net) -> COL1+2
- J1 pad 14: (no net) -> COL5+6
- J1 pad 2: /ROW3+4 -> ROW3
- J1 pad 3: /ROW5+6 -> ROW5
- J1 pad 4: COL1+2 -> Net-(J1-Pad4)
- J1 pad 5: COL3+4 -> Net-(J1-Pad5)
- J1 pad 6: COL5+6 -> COL3+4
- J1 pad 8: arrowsR -> Arrow-Right
- J1 pad 9: arrowsC -> ROW2
- SW1 pad 1: /ROW1+2 -> ROW1
- SW10 pad 1: /ROW5+6 -> ROW5
- SW11 pad 1: /ROW3+4 -> ROW4
- SW12 pad 1: /ROW5+6 -> ROW6
- SW13 pad 1: /ROW1+2 -> ROW1
- SW14 pad 1: /ROW1+2 -> ROW2
- SW15 pad 1: /ROW3+4 -> ROW3
- SW16 pad 1: /ROW5+6 -> ROW5
- SW17 pad 1: /ROW3+4 -> ROW4
- SW18 pad 1: /ROW5+6 -> ROW6
- SW19 pad 1: /ROW1+2 -> ROW1
- SW2 pad 1: /ROW1+2 -> ROW2
- SW20 pad 1: /ROW1+2 -> ROW2
- SW21 pad 1: /ROW3+4 -> ROW3
- SW22 pad 1: /ROW5+6 -> ROW5
- SW23 pad 1: /ROW3+4 -> ROW4
- SW24 pad 1: /ROW5+6 -> ROW6
- SW25 pad 1: /ROW1+2 -> ROW1
- SW26 pad 1: /ROW1+2 -> ROW2
- SW27 pad 1: /ROW3+4 -> ROW3
- SW28 pad 1: /ROW5+6 -> ROW5
- SW29 pad 1: /ROW3+4 -> ROW4
- SW3 pad 1: /ROW3+4 -> ROW3
- SW30 pad 1: /ROW5+6 -> ROW6
- SW31 pad 1: /ROW1+2 -> ROW1
- SW32 pad 1: /ROW1+2 -> ROW2
- SW33 pad 1: /ROW3+4 -> ROW3
- SW34 pad 1: /ROW5+6 -> ROW5
- SW35 pad 1: /ROW3+4 -> ROW4
- SW36 pad 1: /ROW1+2 -> ROW1
- SW37 pad 1: /ROW1+2 -> ROW2
- SW38 pad 1: /ROW3+4 -> ROW3
- SW39 pad 1: /ROW5+6 -> ROW5
- SW4 pad 1: /ROW5+6 -> ROW5
- SW40 pad 1: /ROW3+4 -> ROW4
- SW41 pad 1: /ROW1+2 -> ROW2
- SW42 pad 1: /ROW3+4 -> ROW3
- SW43 pad 1: /ROW5+6 -> ROW5
- SW44 pad 1: arrowsR -> ROW6
- SW45 pad 1: arrowsR -> ROW5
- SW46 pad 1: arrowsR -> ROW6
- SW47 pad 1: arrowsR -> ROW6
- SW5 pad 1: /ROW3+4 -> ROW4
- SW6 pad 1: /ROW5+6 -> ROW6
- SW7 pad 1: /ROW1+2 -> ROW1
- SW8 pad 1: /ROW1+2 -> ROW2
- SW9 pad 1: /ROW3+4 -> ROW3
Routing:
- net /ROW1+2: track 482.8 -> 0.00 mm
- net /ROW3+4: track 424.7 -> 0.00 mm
- net /ROW5+6: track 341.0 -> 0.00 mm
- net ROW1: track 0.00 -> 330.8 mm
- net ROW2: track 0.00 -> 316.0 mm
- net ROW3: track 0.00 -> 281.3 mm
- net ROW4: track 0.00 -> 257.6 mm
- net ROW5: track 0.00 -> 254.9 mm
- net ROW6: track 0.00 -> 224.2 mm
- net arrowsC: track 123.5 -> 0.00 mm
- net arrowsR: track 104.3 -> 0.00 mm
- net Arrow-Right: track 0.00 -> 66.6 mm
- net COL7+8: track 216.9 -> 273.9 mm
- net COL5+6: track 328.3 -> 367.9 mm
- net COL3+4: track 381.7 -> 412.8 mm
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Other:
- board text added: "https://github.com/Supermagnum/98keys-ergo/"

Commit message: Add files via upload
update
Parts:
- J1: value DB15_Female -> 5745783-4; footprint Connector_Dsub:DSUB-15-HD_Female_Horizontal_P2.29x1.98mm_EdgePinOffset3.03mm_Housed_MountingHolesOffset4.94mm -> Connector_Dsub:DSUB-25_Female_Horizontal_P2.77x2.84mm_EdgePinOffset4.94mm_Housed_MountingHolesOffset7.48mm
- moved J1 32.6 mm to (32.0, 159.9)
Connections:
- D1 pad 1: COL1+2 -> COL1
- D10 pad 1: COL1+2 -> COL2
- D11 pad 1: COL1+2 -> COL2
- D12 pad 1: COL1+2 -> COL2
- D14 pad 1: COL3+4 -> COL3
- D15 pad 1: COL3+4 -> COL3
- D16 pad 1: COL3+4 -> COL3
- D17 pad 1: COL3+4 -> COL3
- D18 pad 1: COL3+4 -> COL3
- D19 pad 1: COL3+4 -> COL3
- D2 pad 1: COL1+2 -> COL1
- D20 pad 1: COL3+4 -> COL4
- D21 pad 1: COL3+4 -> COL4
- D22 pad 1: COL3+4 -> COL4
- D23 pad 1: COL3+4 -> COL4
- D24 pad 1: COL3+4 -> COL4
- D25 pad 1: COL3+4 -> COL4
- D26 pad 1: COL5+6 -> COL5
- D27 pad 1: COL5+6 -> COL5
- D28 pad 1: COL5+6 -> COL5
- D29 pad 1: COL5+6 -> COL5
- D3 pad 1: COL1+2 -> COL1
- D30 pad 1: COL5+6 -> COL5
- D31 pad 1: COL5+6 -> COL5
- D32 pad 1: COL5+6 -> COL6
- D33 pad 1: COL5+6 -> COL6
- D34 pad 1: COL5+6 -> COL6
- D35 pad 1: COL5+6 -> COL6
- D36 pad 1: COL5+6 -> COL6
- D37 pad 1: COL7+8 -> COL7
- D38 pad 1: COL7+8 -> COL7
- D39 pad 1: COL7+8 -> COL7
- D4 pad 1: COL1+2 -> COL1
- D40 pad 1: COL7+8 -> COL7
- D41 pad 1: COL7+8 -> COL7
- D42 pad 1: COL7+8 -> COL8
- D43 pad 1: COL7+8 -> COL8
- D44 pad 1: COL7+8 -> COL8
- D45 pad 1: COL5+6 -> COL6
- D47 pad 1: COL7+8 -> COL8
- D5 pad 1: COL1+2 -> COL1
- D6 pad 1: COL1+2 -> COL1
- D7 pad 1: COL1+2 -> COL2
- D8 pad 1: COL1+2 -> COL2
- D9 pad 1: COL1+2 -> COL2
- J1 pad 0: (no net) -> GND
- J1 pad 10: ROW4 -> Net-(J1-Pad10)
- J1 pad 11: ROW6 -> Net-(J1-Pad11)
- J1 pad 13: COL1+2 -> Net-(J1-Pad13)
- J1 pad 14: COL5+6 -> ROW2
- J1 pad 15: GND -> ROW4
- J1 pad 4: Net-(J1-Pad4) -> COL1
- J1 pad 5: Net-(J1-Pad5) -> COL3
- J1 pad 6: COL3+4 -> COL5
- J1 pad 7: COL7+8 -> COL7
- J1 pad 9: ROW2 -> Net-(J1-Pad9)
Routing:
- net COL1+2: track 474.7 -> 0.00 mm
- net COL3+4: track 412.8 -> 0.00 mm
- net COL5+6: track 367.9 -> 0.00 mm
- net COL1: track 0.00 -> 329.9 mm
- net COL2: track 0.00 -> 299.1 mm
- net COL7+8: track 273.9 -> 0.00 mm
- net COL3: track 0.00 -> 269.0 mm
- net COL4: track 0.00 -> 245.8 mm
- net COL6: track 0.00 -> 231.7 mm
- net COL5: track 0.00 -> 225.0 mm
- net COL7: track 0.00 -> 162.8 mm
- net COL8: track 0.00 -> 157.2 mm
- net ROW2: track 316.0 -> 275.7 mm
- net ROW1: track 330.8 -> 296.7 mm
- net ROW4: track 257.6 -> 223.9 mm
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Other:
- net class columns added: clearance 0.2, trace_width 0.25, via_dia 0.8, via_drill 0.4
