File: right/pcb-flat-right.sch (KiCad schematic (older format))
At the start: 103 parts, among them J1 DB15_Female, SW1 MX-NO-LED, SW10 MX-NO-LED, SW11 MX-NO-LED, SW12 MX-NO-LED, SW13 MX-NO-LED, SW14 MX-NO-LED, SW15 MX-NO-LED, SW16 MX-NO-LED, SW17 MX-NO-LED, SW18 MX-NO-LED, SW19 MX-NO-LED, SW2 MX-NO-LED, SW20 MX-NO-LED, SW21 MX-NO-LED, SW22 MX-NO-LED, SW23 MX-NO-LED, SW24 MX-NO-LED, SW25 MX-NO-LED, SW26 MX-NO-LED, SW27 MX-NO-LED, SW28 MX-NO-LED, SW29 MX-NO-LED, SW3 MX-NO-LED, SW30 MX-NO-LED, SW31 MX-NO-LED, SW32 MX-NO-LED, SW33 MX-NO-LED, SW34 MX-NO-LED, SW35 MX-NO-LED, SW36 MX-NO-LED, SW37 MX-NO-LED, SW38 MX-NO-LED, SW39 MX-NO-LED, SW4 MX-NO-LED, SW40 MX-NO-LED, SW41 MX-NO-LED, SW42 MX-NO-LED, SW43 MX-NO-LED, SW44 MX-NO-LED, SW45 MX-NO-LED, SW46 MX-NO-LED, SW47 MX-NO-LED, SW5 MX-NO-LED, SW6 MX-NO-LED, SW7 MX-NO-LED, SW8 MX-NO-LED, SW9 MX-NO-LED

Commit message: updated files, right side.
Parts:
- J1: footprint Connector_Dsub:DSUB-15-HD_Female_Horizontal_P2.29x1.98mm_EdgePinOffset9.40mm -> Connector_Dsub:DSUB-15-HD_Female_Horizontal_P2.29x1.98mm_EdgePinOffset3.03mm_Housed_MountingHolesOffset4.94mm
- SW44: Field4 (none) -> arrow-left
- SW45: Field4 (none) -> arrow-up
- SW46: Field4 (none) -> arrow-down
- SW47: Field4 (none) -> arrow-right
Connections:
- net COL1+2: now also J1.13 (P13); no longer J1.4
- net COL3+4: now also J1.6; no longer J1.5
- net COL5+6: now also D45.1 (K), J1.14 (P14); no longer J1.6
- net COL7+8: now also D47.1 (K)
- net ROW4: now reaches J1.10 (P10)
- net ROW4: now also SW11.1, SW17.1, SW23.1, SW29.1, SW35.1, SW40.1, SW5.1
- net ROW6: now reaches J1.11 (P111)
- net ROW6: now also SW12.1, SW18.1, SW24.1, SW30.1, SW44.1, SW46.1, SW47.1, SW6.1
- removed net ArrowsC: D45.1 (K), D46.1 (K), D47.1 (K), D48.1 (K), J1.9 (P9)
- removed net ArrowsR: J1.8, SW44.1, SW45.1, SW46.1, SW47.1
- net ROW1+2 renamed ROW1
- net ROW1: no longer SW14.1, SW2.1, SW20.1, SW26.1, SW32.1, SW37.1, SW41.1, SW8.1
- net ROW3+4 renamed ROW3
- net ROW3: no longer SW11.1, SW17.1, SW23.1, SW29.1, SW35.1, SW40.1, SW5.1
- net ROW5+6 renamed ROW5
- net ROW5: now also SW45.1; no longer SW12.1, SW18.1, SW24.1, SW30.1, SW6.1
- new net Arrow-Right: D46.1 (K), D48.1 (K), J1.8
- new net ROW2: J1.9 (P9), SW14.1, SW2.1, SW20.1, SW26.1, SW32.1, SW37.1, SW41.1, SW8.1
- no-connect marks 5 -> 3
Other:
- moved on the sheet: D45, D46, D47, D48, H1, H2, H3, H4, H5, H6, H7, H8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

Commit message: Add files via upload
update
Parts:
- removed J1: DB15_Female, Connector_Dsub:DSUB-15-HD_Female_Horizontal_P2.29x1.98mm_EdgePinOffset3.03mm_Housed_MountingHolesOffset4.94mm, symbol Connector:DB15_Female
- added J1: 5745783-4, Connector_Dsub:DSUB-25_Female_Horizontal_P2.77x2.84mm_EdgePinOffset4.94mm_Housed_MountingHolesOffset7.48mm, symbol Connector:DB25_Female_MountingHoles
Connections:
- net labels added: COL1, COL2, COL3, COL4, COL5, COL6, COL7, COL8
- net labels removed: COL1+2, COL3+4, COL5+6, COL7+8
- wire segments 238 -> 242
- no-connect marks 3 -> 10
Changed lines of the file:
@@
 	12350 1350 12350 3800
-Wire Wire Line
-	11000 1350 12350 1350
-Wire Wire Line
-	11000 10300 11000 8400
 Wire Wire Line
 	9500 2400 9500 2350
@@
 $EndComp
 Wire Wire Line
-	9150 1350 10050 1350
-Wire Wire Line
-	9150 10250 9150 9550
-Wire Wire Line
 	8250 3950 8250 5550
 Connection ~ 8250 3950
@@
 $EndComp
 Wire Wire Line
-	7250 1350 8250 1350
-Wire Wire Line
 	8250 1350 8250 2550
-Wire Wire Line
-	7250 10250 7250 9500
 Wire Wire Line
 	6200 9400 6250 9400
@@
 Wire Wire Line
 	6250 1350 6250 2350
-Wire Wire Line
-	5350 1350 6250 1350
 Connection ~ 4750 7550
 Connection ~ 8700 8800
@@
 Text Label 17300 3850 0    50   ~ 0
 GND
-Text GLabel 7250 10250 3    50   BiDi ~ 0
-COL3+4
-Text GLabel 9150 10250 3    50   BiDi ~ 0
-COL5+6
-Text GLabel 11000 10300 3    50   BiDi ~ 0
-COL7+8
 Text GLabel 17000 3850 0    50   Input ~ 0
 GND
-Text GLabel 5350 10400 3    50   Input ~ 0
-COL1+2
-Wire Wire Line
-	5350 9400 5350 10400
-$Comp
-L Connector:DB15_Female J?
-U 1 1 5FA2CB1C
-P 14750 4800
-AR Path="/5F5CF1CF/5FA2CB1C" Ref="J?"  Part="1"
-AR Path="/5FA2CB1C" Ref="J1"  Part="1"
-F 0 "J1" H 14904 4846 50  0000 L CNN
-F 1 "DB15_Female" H 14904 4755 50  0000 L CNN
-F 2 "Connector_Dsub:DSUB-15-HD_Female_Horizontal_P2.29x1.98mm_EdgePinOffset3.03mm_Housed_MountingHolesOffset4.94mm" H 14750 4800 50  0001 C CNN
-F 3 " ~" H 14750 4800 50  0001 C CNN
-	1    14750 4800
-	1    0    0    -1
-$EndComp
 Text GLabel 14000 4100 0    50   Input ~ 0
 ROW1
@@
 Wire Wire Line
 	14450 4500 14000 4500
-Text GLabel 14000 5000 0    50   Input ~ 0
-COL1+2
-Text GLabel 14000 5100 0    50   Input ~ 0
-COL3+4
-Wire Wire Line
-	14450 5000 14000 5000
-Wire Wire Line
-	14000 5100 14450 5100
-Text GLabel 14000 5200 0    50   Input ~ 0
-COL5+6
-Wire Wire Line
-	14450 5200 14000 5200
-Text GLabel 14000 5300 0    50   Input ~ 0
-COL7+8
-Wire Wire Line
-	14450 5300 14000 5300
 Wire Wire Line
 	14450 5500 14000 5500
-Text GLabel 13850 5400 0    50   Input ~ 0
+Text GLabel 14650 6700 0    50   Input ~ 0
 GND
-Wire Wire Line
-	14450 5400 13850 5400
 Wire Wire Line
 	17000 3850 18200 3850
@@
 Text GLabel 14000 5500 0    50   BiDi ~ 0
 Arrow-Right
-NoConn ~ 14450 4700
-NoConn ~ 14450 4800
-NoConn ~ 14450 4900
-Text Label 5350 10050 0    50   ~ 0
-COL1+2
-Text Label 7250 9850 0    50   ~ 0
-COL3+4
-Text Label 9150 9950 0    50   ~ 0
-COL5+6
-Text Label 11000 9900 0    50   ~ 0
-COL7+8
 Text Label 13250 10000 0    50   ~ 0
 Arrow-col
+$Comp
+L Connector:DB25_Female_MountingHoles J1
+U 1 1 5F5F469C
+P 14750 5300
+F 0 "J1" H 14930 5302 50  0000 L CNN
+F 1 "5745783-4 " H 14930 5211 50  0000 L CNN
+F 2 "Connector_Dsub:DSUB-25_Female_Horizontal_P2.77x2.84mm_EdgePinOffset4.94mm_Housed_MountingHolesOffset7.48mm" H 14750 5300 50  0001 C CNN
+F 3 " ~" H 14750 5300 50  0001 C CNN
+F 4 "DB-25-female" H 15250 5150 50  0000 C CNN "Field4"
+	1    14750 5300
+	1    0    0    -1
+$EndComp
+Wire Wire Line
+	14750 6700 14650 6700
+Text GLabel 14000 4700 0    50   Input ~ 0
+COL1
+Text GLabel 14000 4800 0    50   Input ~ 0
+COL2
+Text GLabel 14000 4900 0    50   Input ~ 0
+COL3
+Text GLabel 14000 5000 0    50   Input ~ 0
+COL4
+Text GLabel 14000 5100 0    50   Input ~ 0
+COL5
+Text GLabel 14000 5200 0    50   Input ~ 0
+COL6
+Text GLabel 14000 5300 0    50   Input ~ 0
+COL7
+Text GLabel 14000 5400 0    50   Input ~ 0
+COL8
+Wire Wire Line
+	14000 4700 14450 4700
+Wire Wire Line
+	14450 4800 14000 4800
+Wire Wire Line
+	14000 4900 14450 4900
+Wire Wire Line
+	14450 5000 14000 5000
+Wire Wire Line
+	14000 5100 14450 5100
+Wire Wire Line
+	14450 5200 14000 5200
+Wire Wire Line
+	14000 5300 14450 5300
+Wire Wire Line
+	14450 5400 14000 5400
+Text GLabel 5350 10850 3    50   Input ~ 0
+COL1
+Text GLabel 6250 9850 3    50   Input ~ 0
+COL2
+Text GLabel 7250 10700 3    50   Input ~ 0
+COL3
+Text GLabel 8250 10050 3    50   Input ~ 0
+COL4
+Text GLabel 9150 10700 3    50   Input ~ 0
+COL5
+Text GLabel 10150 9850 3    50   Input ~ 0
+COL6
+Text GLabel 11000 10750 3    50   Input ~ 0
+COL7
+Text GLabel 12350 9850 3    50   Input ~ 0
+COL8
+Wire Wire Line
+	6250 9400 6250 9850
+Wire Wire Line
+	8250 9600 8250 10050
+Wire Wire Line
+	10150 9400 10150 9850
+Wire Wire Line
+	12350 9400 12350 9850
+Wire Wire Line
+	5350 9400 5350 10850
+Connection ~ 6250 9400
+Wire Wire Line
+	7250 9500 7250 10700
+Connection ~ 8250 9600
+Wire Wire Line
+	9150 9550 9150 10700
+Connection ~ 10150 9400
+Wire Wire Line
+	11000 8400 11000 10750
+Connection ~ 12350 9400
+NoConn ~ 14450 5600
+NoConn ~ 14450 5700
+NoConn ~ 14450 5800
+NoConn ~ 14450 5900
+NoConn ~ 14450 6000
+NoConn ~ 14450 6100
+NoConn ~ 14450 6200
+NoConn ~ 14450 6300
+NoConn ~ 14450 6400
+NoConn ~ 14450 6500
 $EndSCHEMATC
