File: 98keys-left/98keys-left.kicad_pcb (KiCad board)
At the start: 2 copper layers, 225.3 x 231.1 mm, 115 parts, among them J1 Conn_01x04_Male, SW1 MX-NO-LED, SW10 MX-NO-LED, SW11 MX-NO-LED, SW12 MX-NO-LED, SW13 MX-NO-LED, SW14 MX-NO-LED, SW15 MX-NO-LED, SW16 MX-NO-LED, SW17 MX-NO-LED, SW18 MX-NO-LED, SW19 MX-NO-LED, SW2 MX-NO-LED, SW20 MX-NO-LED, SW21 MX-NO-LED, SW22 MX-NO-LED, SW23 MX-NO-LED, SW24 MX-NO-LED, SW25 MX-NO-LED, SW26 MX-NO-LED, SW27 MX-NO-LED, SW28 MX-NO-LED, SW29 MX-NO-LED, SW3 MX-NO-LED, SW30 MX-NO-LED, SW31 MX-NO-LED, SW32 MX-NO-LED, SW33 MX-NO-LED, SW34 MX-NO-LED, SW35 MX-NO-LED, SW36 MX-NO-LED, SW37 MX-NO-LED, SW38 MX-NO-LED, SW39 MX-NO-LED, SW4 MX-NO-LED, SW40 MX-NO-LED, SW41 MX-NO-LED, SW42 MX-NO-LED, SW43 MX-NO-LED, SW44 MX-NO-LED, SW45 MX-NO-LED, SW46 MX-NO-LED, SW47 MX-NO-LED, SW48 SW_Push, SW5 MX-NO-LED, SW6 MX-NO-LED, SW7 MX-NO-LED, SW8 MX-NO-LED, SW9 MX-NO-LED, U1 Pico

Commit message: Add files via upload
Parts:
- J1: footprint Connector_PinHeader_2.54mm:PinHeader_1x04_P2.54mm_Vertical -> Connector_Audio:Jack_3.5mm_CUI_SJ1-43514_Horizontal
- moved R6 94.8 mm to (147.0, 51.5), turned to 90 degrees
- moved J1 93.7 mm to (155.5, 47.9), turned to 180 degrees
- moved R5 90.0 mm to (164.0, 46.5), turned to -90 degrees
Connections:
- net SDC I2C0 renamed SCL I2C0
Routing:
- net PWM4: track 69.9 -> 193.5 mm, vias 1 -> 2
- net VCC: track 25.9 -> 108.9 mm, vias 0 -> 1
- net ROW2: track 325.1 -> 261.0 mm, vias 2 -> 1
- net PWM3: track 123.2 -> 72.3 mm, vias 2 -> 1
- net SCL I2C0: track 45.1 -> 93.4 mm
- net SDA I2C0: track 51.3 -> 98.6 mm
- net ROW3: track 337.5 -> 292.2 mm, vias 1 -> 0
- net COL2: track 317.2 -> 351.8 mm
- net PWM1: track 78.1 -> 46.4 mm
- net COL3: track 260.8 -> 292.5 mm, vias 1 -> 0
- net ROW6: track 404.9 -> 434.0 mm
- net ROW4: track 296.9 -> 276.1 mm, vias 1 -> 0
- net ROW1: track 240.4 -> 222.1 mm, vias 1 -> 0
- net COL8: track 255.7 -> 273.1 mm, vias 2 -> 1
- net ROW5: track 366.4 -> 378.5 mm, vias 0 -> 1
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Other:
- outline, holes or cut-outs redrawn
