File: 98keys-right/98keys-right.kicad_sch (KiCad schematic)
At the start: 115 parts, among them J1 Conn_01x04_Male/I2C, SW1 MX-NO-LED, SW10 MX-NO-LED, SW11 MX-NO-LED, SW12 MX-NO-LED, SW13 MX-NO-LED, SW14 MX-NO-LED, SW15 MX-NO-LED, SW16 MX-NO-LED, SW17 MX-NO-LED, SW18 MX-NO-LED, SW19 MX-NO-LED, SW2 MX-NO-LED, SW20 MX-NO-LED, SW21 MX-NO-LED, SW22 MX-NO-LED, SW23 MX-NO-LED, SW24 MX-NO-LED, SW25 MX-NO-LED, SW26 MX-NO-LED, SW27 MX-NO-LED, SW28 MX-NO-LED, SW29 MX-NO-LED, SW3 MX-NO-LED, SW30 MX-NO-LED, SW31 MX-NO-LED, SW32 MX-NO-LED, SW33 MX-NO-LED, SW34 MX-NO-LED, SW35 MX-NO-LED, SW36 MX-NO-LED, SW37 MX-NO-LED, SW38 MX-NO-LED, SW39 MX-NO-LED, SW4 MX-NO-LED, SW40 MX-NO-LED, SW41 MX-NO-LED, SW42 MX-NO-LED, SW43 MX-NO-LED, SW44 MX-NO-LED, SW45 MX-NO-LED, SW46 MX-NO-LED, SW47 MX-NO-LED, SW48 SW_Push/KS-01Q-01, SW5 MX-NO-LED, SW6 MX-NO-LED, SW7 MX-NO-LED, SW8 MX-NO-LED, SW9 MX-NO-LED, U1 Pico

Commit message: Add files via upload
Parts:
- J1: footprint Connector_PinHeader_2.54mm:PinHeader_1x04_P2.54mm_Vertical -> Connector_Audio:Jack_3.5mm_CUI_SJ1-43514_Horizontal
Changed lines of the file:
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@@
     (property "Reference" "J1" (id 0) (at 384.175 130.81 0))
     (property "Value" "Conn_01x04_Male/I2C" (id 1) (at 384.175 133.35 0))
-    (property "Footprint" "Connector_PinHeader_2.54mm:PinHeader_1x04_P2.54mm_Vertical" (id 2) (at 383.54 138.43 0)
+    (property "Footprint" "Connector_Audio:Jack_3.5mm_CUI_SJ1-43514_Horizontal" (id 2) (at 383.54 138.43 0)
       (effects (font (size 1.27 1.27)) hide)
     )
@@
     )
     (path "/bcbf6456-a268-4571-98a7-f76d400f1e35"
-      (reference "J1") (unit 1) (value "Conn_01x04_Male/I2C") (footprint "Connector_PinHeader_2.54mm:PinHeader_1x04_P2.54mm_Vertical")
+      (reference "J1") (unit 1) (value "Conn_01x04_Male/I2C") (footprint "Connector_Audio:Jack_3.5mm_CUI_SJ1-43514_Horizontal")
     )
     (path "/60fbabbc-1e62-457b-9c32-9706b1a8627e"
