File: 98keys-split-pcb/98keys-split-pcb.kicad_sch (KiCad schematic)
At the start: 230 parts, among them J1 Conn_01x04_Male/I2C, J2 Conn_01x04_Male, SW1 MX-NO-LED, SW10 MX-NO-LED, SW11 MX-NO-LED, SW12 MX-NO-LED, SW13 MX-NO-LED, SW14 MX-NO-LED, SW15 MX-NO-LED, SW16 MX-NO-LED, SW17 MX-NO-LED, SW18 MX-NO-LED, SW19 MX-NO-LED, SW2 MX-NO-LED, SW20 MX-NO-LED, SW21 MX-NO-LED, SW22 MX-NO-LED, SW23 MX-NO-LED, SW24 MX-NO-LED, SW25 MX-NO-LED, SW26 MX-NO-LED, SW27 MX-NO-LED, SW28 MX-NO-LED, SW29 MX-NO-LED, SW3 MX-NO-LED, SW30 MX-NO-LED, SW31 MX-NO-LED, SW32 MX-NO-LED, SW33 MX-NO-LED, SW34 MX-NO-LED, SW35 MX-NO-LED, SW36 MX-NO-LED, SW37 MX-NO-LED, SW38 MX-NO-LED, SW39 MX-NO-LED, SW4 MX-NO-LED, SW40 MX-NO-LED, SW41 MX-NO-LED, SW42 MX-NO-LED, SW43 MX-NO-LED, SW44 MX-NO-LED, SW45 MX-NO-LED, SW46 MX-NO-LED, SW47 MX-NO-LED, SW48 SW_Push/KS-01Q-01, SW49 SW_Push, SW5 MX-NO-LED, SW50 MX-NO-LED, SW51 MX-NO-LED, SW52 MX-NO-LED, SW53 MX-NO-LED, SW54 MX-NO-LED, SW55 MX-NO-LED, SW56 MX-NO-LED, SW57 MX-NO-LED, SW58 MX-NO-LED, SW59 MX-NO-LED, SW6 MX-NO-LED, SW60 MX-NO-LED, SW61 MX-NO-LED, SW62 MX-NO-LED, SW63 MX-NO-LED, SW64 MX-NO-LED, SW65 MX-NO-LED, SW66 MX-NO-LED, SW67 MX-NO-LED, SW68 MX-NO-LED, SW69 MX-NO-LED, SW7 MX-NO-LED, SW70 MX-NO-LED, SW71 MX-NO-LED, SW72 MX-NO-LED, SW73 MX-NO-LED, SW74 MX-NO-LED, SW75 MX-NO-LED, SW76 MX-NO-LED, SW77 MX-NO-LED, SW78 MX-NO-LED, SW79 MX-NO-LED, SW8 MX-NO-LED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

Commit message: Updated pcb files.
Parts:
- SW48: value SW_Push/KS-01Q-01 -> SW_Push; footprint Button_Switch_THT:Push_E-Switch_KS01Q01 -> switch:switch_P5.08mm
- SW49: footprint Button_Switch_THT:Push_E-Switch_KS01Q01 -> switch:switch_P5.08mm
Other:
- note added: "CAPS"
- note added: "EG2614-ND"
- note added: "Keyswitch Hotswap sockets: 0305-2-15-80-47-80-10-0 or Digikey: ED90584-ND"
- note added: "L1"
- note added: "L2"
- note added: "OMIT R9 R11 IF SERIAL COMM IS USED."
- note added: "Scroll"
- note added: "TRRS jack, SJ1-42514"
- moved on the sheet: D48, D49, D50, D51, D52, D53, D54, D55, J1, J2, R1, R10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
